File: Hardware/mightIO_tile.brd (EAGLE design)
At the start: 76.5 x 63.5 mm, 188 parts, among them IC1 TL064D, IC10 TL064D, IC11 TL064D, IC12 LM4041A12DBZ, IC2 TL064D, IC3 LM4041A12DBZ, IC4 TL064D, IC5 TL064D, IC6 LM4041A12DBZ, IC7 TL064D, IC8 TL064D, IC9 LM4041A12DBZ, U1 MAX11612, U2 MAX11612, U3 MAX11612, U4 MAX11612

Commit message: Updated tiled board
Parts:
- added C69: 47pF, rcl:C0603
- added C70, C72: 0.1uF, rcl:C0603
- added C71: 10uF, rcl:E2,5-6
- added JP13, JP14, JP15: (no value), pinhead:1X04
- added JP16: (no value), pinhead:1X03
- C21, C38, C39, C55, C56, C57: value 2.2uF -> 0.1uF
- C25, C42, C59: value 220pF -> 2.2uF
- C26, C29, C32, C44, C49: value 47pF -> 220pF
- C28, C30, C45, C48, C64: value 220pF -> 47pF
- C33: value 0.1uF -> 47pF
- C34: value 10uF -> 0.1uF; device rcl:E2,5-6 -> rcl:C0603
- C35, C53: value 0.1uF -> 10uF; device rcl:C0603 -> rcl:E2,5-6
- C43, C60, C61: value 47pF -> 2.2uF
- C50, C67: value 0.1uF -> 220pF
- C51: value 10uF -> 47pF; device rcl:E2,5-6 -> rcl:C0603
- C68: value 10uF -> 220pF; device rcl:E2,5-6 -> rcl:C0603
- JP1, JP10, JP7: value Apple -> (none)
- JP11, JP3, JP5: value Banana -> (none)
- JP12: value Mango -> (none); device pinhead:1X04 -> pinhead:1X03
- JP2: value Apple -> (none); device pinhead:1X04 -> pinhead:1X03
- JP4, JP6, JP9: value Mango -> (none)
- JP8: value Banana -> (none); device pinhead:1X04 -> pinhead:1X03
- R11, R19, R26, R28, R32, R38, R47, R49, R5, R53, R59, R68, R7, R70, R74, R80: value 20k -> 22k
- R16, R41, R62, R83: value 2k -> 1k
- R21, R42, R63, R84: value 10k -> 5.1k
- moved C28 71.6 mm to (70.8, 14.0), turned to 270 degrees
- moved C30 71.5 mm to (72.7, 14.0), flipped to the top
- moved JP5 66.9 mm to (51.1, 6.35), turned to 0 degrees
- moved C37 64.5 mm to (5.40, 45.7), flipped to the bottom, turned to 0 degrees
- moved C44 63.0 mm to (13.7, 57.1), flipped to the top, turned to 90 degrees
- moved C51 62.4 mm to (28.3, 59.1), flipped to the bottom, turned to 90 degrees
- moved JP9 61.2 mm to (13.0, 38.1), turned to 0 degrees
- moved C25 60.9 mm to (55.6, 13.0), flipped to the bottom, turned to 270 degrees
- moved C50 60.3 mm to (13.7, 50.8), turned to 270 degrees
- moved C20 59.3 mm to (69.2, 8.26), flipped to the bottom, turned to 180 degrees
- moved R59 58.8 mm to (27.9, 56.2), turned to 180 degrees
- moved C49 58.2 mm to (11.4, 50.8), turned to 270 degrees
- moved C21 57.8 mm to (58.1, 9.53), turned to 270 degrees
- moved R47 57.3 mm to (27.9, 56.2), flipped to the top, turned to 0 degrees
- moved C40 56.2 mm to (14.9, 47.9), turned to 180 degrees
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Connections:
- removed net N$81: C59.2, IC10.1, R67.1, U4.P$1
- removed net N$82: C64.2, IC11.1, R77.1, U4.P$3
- removed net N$83: C65.2, IC10.7, R79.1, U4.P$4
- removed net N$84: R70.2, U$8.P$6
- removed net VREF: C14.2, IC1.10, IC1.12, IC1.3, IC1.5, IC2.10, IC2.12, IC2.3, IC2.5, R16.2, R21.1
- removed net VREF1: C33.2, IC4.10, IC4.12, IC4.3, IC4.5, IC5.10, IC5.12, IC5.3, IC5.5, R41.2, R42.1
- removed net VREF2: C50.2, IC7.10, IC7.12, IC7.3, IC7.5, IC8.10, IC8.12, IC8.3, IC8.5, R62.2, R63.1
- removed net VREF3: C67.2, IC10.10, IC10.12, IC10.3, IC10.5, IC11.10, IC11.12, IC11.3, IC11.5, R83.2, R84.1
- new net VREFIN: C14.1, IC1.3, IC1.5, IC2.3, IC2.5, R16.2, R21.1
- new net VREFIN1: C34.1, IC4.3, IC4.5, IC5.3, IC5.5, R41.2, R42.1
- new net VREFIN2: C52.1, IC7.3, IC7.5, IC8.3, IC8.5, R62.2, R63.1
- new net VREFIN3: C70.1, IC10.3, IC10.5, IC11.3, IC11.5, R83.2, R84.1
- new net VREFOUT: C18.1, IC3.1, R11.2, R15.1, R16.1, R19.2, R5.2, R7.2
- new net VREFOUT1: C36.1, IC6.1, R26.2, R28.2, R32.2, R38.2, R40.1, R41.1
- new net VREFOUT2: C54.1, IC9.1, R47.2, R49.2, R53.2, R59.2, R61.1, R62.1
- new net VREFOUT3: C72.1, IC12.1, R68.2, R70.2, R74.2, R80.2, R82.1, R83.1
- net +5V: now also C1.1, C2.1, C3.1; no longer C1.2, C2.2, C3.2
- net +5V1: now also C19.1, C20.1, C21.1, C24.2, C35.+, JP5.3; no longer C18.2, C19.2, C20.2, C23.2, C34.+, JP2.3
- net +5V2: now also C37.1, C38.1, C39.1, C42.2, C53.+, JP9.3; no longer C35.2, C36.2, C37.2, C40.2, C51.+, JP7.3
- net +5V3: now also C55.1, C56.1, C57.1, C60.2, C71.+, JP13.3; no longer C52.2, C53.2, C54.2, C57.2, C68.+, JP10.3
- net AI10: now also JP10.1; no longer JP8.1
- net AI11: now also JP10.2; no longer JP8.2
- net AI12: now also JP14.3; no longer JP11.3
- net AI13: now also JP14.4; no longer JP11.4
- net AI14: now also JP14.1; no longer JP11.1
- net AI15: now also JP14.2; no longer JP11.2
- net AI4: now also JP6.3; no longer JP5.3
- net AI5: now also JP6.4; no longer JP5.4
- net AI6: now also JP6.1; no longer JP5.1
- net AI7: now also JP6.2; no longer JP5.2
- net AI8: now also JP10.3; no longer JP8.3
- net AI9: now also JP10.4; no longer JP8.4
- net AOA: now also C10.1; no longer C10.2
- net AOA1: now also C28.1, JP7.1; no longer C27.2, JP6.1
- net AOA2: now also C46.1, JP11.1; no longer C44.2, JP9.1
- net AOA3: now also C64.1, JP15.1; no longer C61.2, JP12.1
- net AOB: now also C12.1; no longer C12.2
- net AOB1: now also C30.1, JP7.2; no longer C29.2, JP6.2
- net AOB2: now also C48.1, JP11.2; no longer C46.2, JP9.2
- net AOB3: now also C66.1, JP15.2; no longer C63.2, JP12.2
- net AOC: now also C9.1; no longer C9.2
- net AOC1: now also C27.1, JP7.3; no longer C26.2, JP6.3
- net AOC2: now also C45.1, JP11.3; no longer C43.2, JP9.3
- net AOC3: now also C63.1, JP15.3; no longer C60.2, JP12.3
- net AOD: now also C16.1; no longer C16.2
- net AOD1: now also C33.1, JP7.4; no longer C32.2, JP6.4
- net AOD2: now also C51.1, JP11.4; no longer C49.2, JP9.4
- net AOD3: now also C69.1, JP15.4; no longer C66.2, JP12.4
- net GND: now also C1.2, C10.2, C12.2, C14.2, C16.2, C18.2, C2.2, C3.2, C9.2, JP2.2; no longer C1.1, C14.1, C2.1, C3.1
- net GND1: now also C19.2, C20.2, C21.2, C25.1, C27.2, C28.2, C30.2, C33.2, C34.2, C35.-, C36.2, JP5.4, JP8.2; no longer C18.1, C19.1, C20.1, C24.1, C33.1, C34.-, JP2.4
- net GND2: now also C37.2, C38.2, C39.2, C43.1, C45.2, C46.2, C48.2, C51.2, C52.2, C53.-, C54.2, JP12.2, JP9.4; no longer C35.1, C36.1, C37.1, C41.1, C50.1, C51.-, JP7.4
- net GND3: now also C55.2, C56.2, C57.2, C61.1, C63.2, C64.2, C66.2, C69.2, C70.2, C71.-, C72.2, JP13.4, JP16.2; no longer C52.1, C53.1, C54.1, C58.1, C67.1, C68.-, JP10.4
- net N$1: now also IC2.10; no longer R19.2
- net N$13: now also IC5.10, U$4.P$9; no longer C22.2, U$3.P$4
- net N$14: now also C22.1, U$3.P$16; no longer C25.1, IC4.2, R24.1, R25.2
- net N$15: now also C22.2, U$3.P$1; no longer C9.1, IC1.13, R5.1, R6.2
- net N$16: now also C23.1, U$3.P$2; no longer C26.1, IC4.13, R26.1, R27.2
- net N$17: now also C23.2, U$3.P$4; no longer C10.1, IC2.13, R7.1, R8.2
- net N$2: now also IC2.9, R19.1, R20.2; no longer R38.2, U$4.P$9
- net N$21: now also C26.1, IC4.2, R24.1, R25.2; no longer C12.1, IC1.9, R11.1, R12.2
- net N$24: now also C29.1, IC5.6, R30.1, R31.2; no longer C27.1, IC5.13, R28.1, R29.2
- net N$25: now also IC2.12; no longer R7.2
- net N$26: now also C31.1, IC5.2, R34.1, R35.2; no longer IC3.1, R15.1, R16.1
- net N$28: now also C32.1, IC4.6, R36.1, R37.2; no longer C28.1, IC5.6, R30.1, R31.2
- net N$29: now also IC4.12, U$4.P$8; no longer C16.1, IC2.9, R19.1, R20.2
- net N$3: now also IC1.10; no longer R11.2
- net N$30: now also C29.2, IC5.7, R31.1, U2.P$2; no longer C29.1, IC4.9, R32.1, R33.2
- net N$31: now also IC4.10, U$4.P$7; no longer C30.1, IC5.2, R34.1, R35.2
- net N$32: now also C26.2, IC4.1, R25.1, U2.P$1; no longer C31.1, IC4.6, R36.1, R37.2
- net N$33: now also C31.2, IC5.1, R35.1, U2.P$3; no longer C32.1, IC5.9, R38.1, R39.2
- net N$34: now also IC1.12; no longer R5.2
- net N$35: now also C32.2, IC4.7, R37.1, U2.P$4; no longer IC6.1, R40.1, R41.1
- net N$36: now also IC5.12, U$4.P$6; no longer R26.2, U$4.P$8
- net N$37: now also IC5.9, R38.1, R39.2; no longer C28.2, IC5.7, R31.1, U2.P$2
- net N$38: now also IC4.13, R26.1, R27.2; no longer R32.2, U$4.P$7
- net N$39: now also IC4.9, R32.1, R33.2; no longer C25.2, IC4.1, R25.1, U2.P$1
- net N$4: now also IC1.13, R5.1, R6.2; no longer C21.1, U$3.P$16
- net N$40: now also IC5.13, R28.1, R29.2; no longer C30.2, IC5.1, R35.1, U2.P$3
- net N$41: now also IC8.10, U$6.P$9; no longer C31.2, IC4.7, R37.1, U2.P$4
- net N$42: now also C40.1, U$5.P$16; no longer R28.2, U$4.P$6
- net N$43: now also C40.2, U$5.P$1; no longer R59.2, U$6.P$9
- net N$44: now also C41.1, U$5.P$2; no longer C38.1, U$5.P$16
- net N$45: now also C41.2, U$5.P$4; no longer C38.2, U$5.P$1
- net N$46: now also C44.1, IC7.2, R45.1, R46.2; no longer C39.1, U$5.P$2
- net N$47: now also C47.1, IC8.6, R51.1, R52.2; no longer C39.2, U$5.P$4
- net N$48: now also C49.1, IC8.2, R55.1, R56.2; no longer C42.1, IC7.2, R45.1, R46.2
- net N$49: now also C50.1, IC7.6, R57.1, R58.2; no longer C43.1, IC7.13, R47.1, R48.2
- net N$5: now also IC1.9, R11.1, R12.2; no longer C21.2, U$3.P$1
- net N$50: now also IC7.12, U$6.P$8; no longer C44.1, IC8.13, R49.1, R50.2
- net N$51: now also C47.2, IC8.7, R52.1, U3.P$2; no longer C45.1, IC8.6, R51.1, R52.2
- net N$52: now also IC7.10, U$6.P$7; no longer C46.1, IC7.9, R53.1, R54.2
- net N$53: now also C44.2, IC7.1, R46.1, U3.P$1; no longer C47.1, IC8.2, R55.1, R56.2
- net N$54: now also C49.2, IC8.1, R56.1, U3.P$3; no longer C48.1, IC7.6, R57.1, R58.2
- net N$55: now also C50.2, IC7.7, R58.1, U3.P$4; no longer C49.1, IC8.9, R59.1, R60.2
- net N$56: now also IC8.12, U$6.P$6; no longer IC9.1, R61.1, R62.1
- net N$57: now also IC8.9, R59.1, R60.2; no longer R47.2, U$6.P$8
- net N$58: now also IC7.13, R47.1, R48.2; no longer C45.2, IC8.7, R52.1, U3.P$2
- net N$59: now also IC7.9, R53.1, R54.2; no longer R53.2, U$6.P$7
- net N$6: now also IC2.13, R7.1, R8.2; no longer C22.1, U$3.P$2
- net N$60: now also IC8.13, R49.1, R50.2; no longer C42.2, IC7.1, R46.1, U3.P$1
- net N$61: now also IC11.10, U$8.P$9; no longer C47.2, IC8.1, R56.1, U3.P$3
- net N$62: now also C58.1, U$7.P$16; no longer C48.2, IC7.7, R58.1, U3.P$4
- net N$63: now also C58.2, U$7.P$1; no longer R49.2, U$6.P$6
- net N$64: now also C59.1, U$7.P$2; no longer R80.2, U$8.P$9
- net N$65: now also C59.2, U$7.P$4; no longer C55.1, U$7.P$16
- net N$66: now also C62.1, IC10.2, R66.1, R67.2; no longer C55.2, U$7.P$1
- net N$67: now also C65.1, IC11.6, R72.1, R73.2; no longer C56.1, U$7.P$2
- net N$68: now also C67.1, IC11.2, R76.1, R77.2; no longer C56.2, U$7.P$4
- net N$69: now also C68.1, IC10.6, R78.1, R79.2; no longer C59.1, IC10.2, R66.1, R67.2
- net N$70: now also IC10.12, U$8.P$8; no longer C60.1, IC10.13, R68.1, R69.2
- net N$71: now also C65.2, IC11.7, R73.1, U4.P$2; no longer C61.1, IC11.13, R70.1, R71.2
- net N$72: now also IC10.10, U$8.P$7; no longer C62.1, IC11.6, R72.1, R73.2
- net N$73: now also C62.2, IC10.1, R67.1, U4.P$1; no longer C63.1, IC10.9, R74.1, R75.2
- net N$74: now also C67.2, IC11.1, R77.1, U4.P$3; no longer C64.1, IC11.2, R76.1, R77.2
- net N$75: now also C68.2, IC10.7, R79.1, U4.P$4; no longer C65.1, IC10.6, R78.1, R79.2
- net N$76: now also IC11.12, U$8.P$6; no longer C66.1, IC11.9, R80.1, R81.2
- net N$77: now also IC11.9, R80.1, R81.2; no longer IC12.1, R82.1, R83.1
- net N$78: now also IC10.13, R68.1, R69.2; no longer R68.2, U$8.P$8
- net N$79: now also IC10.9, R74.1, R75.2; no longer C62.2, IC11.7, R73.1, U4.P$2
- net N$80: now also IC11.13, R70.1, R71.2; no longer R74.2, U$8.P$7
- net SCL1: now also JP5.1; no longer JP2.1
- net SCL2: now also JP9.1; no longer JP7.1
- net SCL3: now also JP13.1; no longer JP10.1
- net SDA1: now also JP5.2; no longer JP2.2
- net SDA2: now also JP9.2; no longer JP7.2
- net SDA3: now also JP13.2; no longer JP10.2
- net V+: now also JP2.1
- net V+1: now also C24.1, JP8.1; no longer C23.1
- net V+2: now also C42.1, JP12.1; no longer C40.1
- net V+3: now also C60.1, JP16.1; no longer C57.1
- net V-: now also JP2.3
- net V-1: now also C25.2, JP8.3; no longer C24.2
- net V-2: now also C43.2, JP12.3; no longer C41.2
- net V-3: now also C61.2, JP16.3; no longer C58.2
Routing:
- net VREF2: track 44.7 -> 0.00 mm, vias 2 -> 0
- net VREF: track 44.7 -> 0.00 mm, vias 2 -> 0
- net VREF3: track 44.7 -> 0.00 mm, vias 2 -> 0
- net VREF1: track 44.7 -> 0.00 mm, vias 2 -> 0
- net VREFOUT: track 0.00 -> 34.8 mm, vias 0 -> 3
- net VREFOUT2: track 0.00 -> 34.8 mm, vias 0 -> 3
- net VREFOUT1: track 0.00 -> 34.8 mm, vias 0 -> 3
- net VREFOUT3: track 0.00 -> 34.8 mm, vias 0 -> 3
- net VREFIN: track 0.00 -> 30.4 mm, vias 0 -> 1
- net VREFIN2: track 0.00 -> 30.4 mm, vias 0 -> 1
- net VREFIN1: track 0.00 -> 30.4 mm, vias 0 -> 1
- net VREFIN3: track 0.00 -> 30.4 mm, vias 0 -> 1
- net N$81: track 19.2 -> 0.00 mm, vias 1 -> 0
- net N$16: track 19.1 -> 2.20 mm, vias 1 -> 0
- net N$82: track 16.2 -> 0.00 mm
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Other:
- board size 76.5 x 63.5 mm -> 75.9 x 63.5 mm
- board text added: "V+"
- board text added: "V-"
