File: Hardware/mightIO.brd (EAGLE design)
At the start: 37.8 x 31.7 mm, 48 parts, among them IC1 TL064D, IC2 TL064D, IC3 LM4041A12DBZ, U1 MAX11612

Commit message: Touched up silkscreen, moved caps
Parts:
- added JP2: (no value), pinhead:1X03
- moved C10 22.5 mm to (32.7, 14.0)
- moved C12 19.8 mm to (34.6, 14.0)
- moved C16 10.3 mm to (28.3, 27.3)
- moved C9 8.47 mm to (28.3, 27.3)
Connections:
- net AOA: now also C10.1
- net AOB: now also C12.1
- net AOC: now also C9.1
- net AOD: now also C16.1
- net GND: now also C10.2, C12.2, C16.2, C9.2, JP2.2
- net V+: now also JP2.1
- net V-: now also JP2.3
Routing:
- net AOB: track 12.7 -> 21.0 mm
- net V+: track 15.6 -> 23.7 mm
- net V-: track 21.4 -> 29.5 mm
- net AOA: track 15.0 -> 18.8 mm
- net AOD: track 11.6 -> 12.3 mm
Other:
- board text added: "V+"
- board text added: "V-"
Changed lines of the file:
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@@
 <text x="32.0675" y="15.24" size="1.016" layer="21" font="vector" ratio="20">AO3</text>
 <wire x1="0" y1="0" x2="37.7825" y2="0" width="0" layer="20"/>
+<text x="25.0825" y="28.575" size="1.016" layer="21" font="vector" ratio="20" rot="R90">V-</text>
+<text x="14.605" y="28.575" size="1.016" layer="21" font="vector" ratio="20" rot="R90">V+</text>
 </plain>
 <attributes>
@@
 <element name="R5" library="rcl" package="R0603" value="22k" x="27.94" y="24.4475"/>
 <element name="R6" library="rcl" package="R0603" value="100k" x="25.4" y="25.4" rot="R270"/>
-<element name="C9" library="rcl" package="C0603" value="47pF" x="20.0025" y="29.21" rot="R90"/>
+<element name="C9" library="rcl" package="C0603" value="47pF" x="28.2575" y="27.305" rot="R90"/>
 <element name="R7" library="rcl" package="R0603" value="22k" x="25.7175" y="14.605" rot="MR270"/>
 <element name="R8" library="rcl" package="R0603" value="100k" x="25.4" y="19.05" rot="MR90"/>
-<element name="C10" library="rcl" package="C0603" value="47pF" x="16.1925" y="29.21" rot="MR270"/>
+<element name="C10" library="rcl" package="C0603" value="47pF" x="32.7025" y="13.97" rot="MR270"/>
 <element name="R9" library="rcl" package="R0603" value="100k" x="7.62" y="23.495" rot="R180"/>
 <element name="R10" library="rcl" package="R0603" value="20k" x="11.43" y="25.4" rot="MR270"/>
@@
 <element name="R11" library="rcl" package="R0603" value="22k" x="27.94" y="20.0025"/>
 <element name="R12" library="rcl" package="R0603" value="100k" x="25.4" y="19.05" rot="R90"/>
-<element name="C12" library="rcl" package="C0603" value="47pF" x="21.9075" y="29.21" rot="R270"/>
+<element name="C12" library="rcl" package="C0603" value="47pF" x="34.6075" y="13.97" rot="R270"/>
 <element name="R13" library="rcl" package="R0603" value="100k" x="7.62" y="20.955" rot="R180"/>
 <element name="R14" library="rcl" package="R0603" value="20k" x="13.6525" y="19.05" rot="MR90"/>
@@
 <element name="R19" library="rcl" package="R0603" value="22k" x="27.94" y="24.4475" rot="MR180"/>
 <element name="R20" library="rcl" package="R0603" value="100k" x="25.4" y="25.4" rot="MR270"/>
-<element name="C16" library="rcl" package="C0603" value="47pF" x="18.0975" y="29.21" rot="MR90"/>
+<element name="C16" library="rcl" package="C0603" value="47pF" x="28.2575" y="27.305" rot="MR90"/>
 <element name="IC3" library="texas" package="DBZ_R-PDSO-G3" value="LM4041A12DBZ" x="29.21" y="11.1125" rot="R270">
 <attribute name="OC_NEWARK" value="58K5875" x="16.51" y="-14.2875" size="1.778" layer="27" rot="R270" display="off"/>
@@
 <element name="C17" library="rcl" package="E2,5-6" value="10uF" x="21.9075" y="5.715" rot="R180"/>
 <element name="C18" library="rcl" package="C0603" value="0.1uF" x="26.035" y="9.525" rot="R270"/>
+<element name="JP2" library="pinhead" package="1X03" value="" x="19.3675" y="29.21"/>
 </elements>
 <signals>
@@
 <contactref element="C17" pad="-"/>
 <contactref element="C3" pad="2"/>
+<contactref element="C16" pad="2"/>
+<contactref element="C9" pad="2"/>
+<contactref element="C12" pad="2"/>
+<contactref element="C10" pad="2"/>
+<contactref element="JP2" pad="2"/>
+<via x="25.7175" y="5.715" extent="1-16" drill="0.6" shape="square"/>
 </signal>
 <signal name="+5V" class="1">
@@
 <wire x1="18.7325" y1="15.24" x2="20.0025" y2="13.97" width="0.4064" layer="1"/>
 <wire x1="20.0025" y1="13.97" x2="20.0025" y2="13.55" width="0.4064" layer="1"/>
+<contactref element="JP2" pad="1"/>
+<wire x1="16.8275" y1="29.21" x2="16.8275" y2="27.6225" width="0.4064" layer="1"/>
+<wire x1="16.8275" y1="27.6225" x2="17.145" y2="27.305" width="0.4064" layer="1"/>
+<wire x1="17.145" y1="27.305" x2="17.78" y2="27.305" width="0.4064" layer="1"/>
+<wire x1="17.78" y1="27.305" x2="18.7325" y2="26.3525" width="0.4064" layer="1"/>
+<wire x1="18.7325" y1="26.3525" x2="18.7325" y2="22.225" width="0.4064" layer="1"/>
 </signal>
 <signal name="N$11">
@@
 <wire x1="18.7325" y1="12.065" x2="20.0025" y2="13.335" width="0.4064" layer="16"/>
 <wire x1="17.4625" y1="12.1675" x2="17.4625" y2="12.065" width="0.4064" layer="16"/>
+<contactref element="JP2" pad="3"/>
+<wire x1="21.9075" y1="29.21" x2="21.9075" y2="27.6225" width="0.4064" layer="1"/>
+<wire x1="21.9075" y1="27.6225" x2="21.59" y2="27.305" width="0.4064" layer="1"/>
+<wire x1="21.59" y1="27.305" x2="20.955" y2="27.305" width="0.4064" layer="1"/>
+<wire x1="20.955" y1="27.305" x2="20.0025" y2="26.3525" width="0.4064" layer="1"/>
+<wire x1="20.0025" y1="26.3525" x2="20.0025" y2="22.225" width="0.4064" layer="1"/>
 </signal>
 <signal name="AI1">
@@
 <wire x1="23.8125" y1="18.415" x2="25.4" y2="18.415" width="0.3048" layer="16"/>
 <wire x1="25.4" y1="18.415" x2="25.4" y2="18.2" width="0.3048" layer="16"/>
+<contactref element="C10" pad="1"/>
+<wire x1="32.7025" y1="14.82" x2="32.7025" y2="16.1925" width="0.3048" layer="16"/>
+<wire x1="32.7025" y1="16.1925" x2="33.3375" y2="16.8275" width="0.3048" layer="16"/>
+<wire x1="33.3375" y1="16.8275" x2="33.3375" y2="18.415" width="0.3048" layer="16"/>
 </signal>
 <signal name="AI3">
@@
 <contactref element="JP4" pad="3"/>
 <wire x1="33.3375" y1="23.495" x2="31.4325" y2="23.495" width="0.3048" layer="1"/>
-<wire x1="30.1625" y1="26.3525" x2="25.5025" y2="26.3525" width="0.3048" layer="1"/>
+<wire x1="30.1625" y1="26.3525" x2="28.575" y2="26.3525" width="0.3048" layer="1"/>
 <contactref element="R6" pad="1"/>
+<wire x1="28.575" y1="26.3525" x2="25.5025" y2="26.3525" width="0.3048" layer="1"/>
 <wire x1="25.4" y1="26.035" x2="25.4" y2="26.25" width="0.3048" layer="1"/>
 <wire x1="30.1625" y1="26.3525" x2="30.48" y2="26.035" width="0.3048" layer="1"/>
@@
 <wire x1="30.48" y1="24.4475" x2="31.4325" y2="23.495" width="0.3048" layer="1"/>
 <wire x1="25.4" y1="26.25" x2="25.5025" y2="26.3525" width="0.3048" layer="1"/>
+<contactref element="C9" pad="1"/>
+<wire x1="28.2575" y1="26.455" x2="28.575" y2="26.455" width="0.3048" layer="1"/>
+<wire x1="28.575" y1="26.455" x2="28.575" y2="26.3525" width="0.3048" layer="1"/>
 </signal>
 <signal name="AOD">
@@
 <contactref element="JP4" pad="4"/>
 <contactref element="R20" pad="1"/>
-<wire x1="33.3375" y1="26.035" x2="25.4" y2="26.035" width="0.3048" layer="16"/>
+<wire x1="33.3375" y1="26.035" x2="27.94" y2="26.035" width="0.3048" layer="16"/>
+<wire x1="27.94" y1="26.035" x2="25.4" y2="26.035" width="0.3048" layer="16"/>
 <wire x1="25.4" y1="26.035" x2="25.4" y2="26.25" width="0.3048" layer="16"/>
+<contactref element="C16" pad="1"/>
+<wire x1="28.2575" y1="26.455" x2="27.94" y2="26.455" width="0.3048" layer="16"/>
+<wire x1="27.94" y1="26.455" x2="27.94" y2="26.035" width="0.3048" layer="16"/>
 </signal>
 <signal name="N$20">
@@
 <wire x1="25.4" y1="18.2" x2="28.6775" y2="18.2" width="0.3048" layer="1"/>
 <wire x1="25.4" y1="18.415" x2="25.4" y2="18.2" width="0.3048" layer="1"/>
+<contactref element="C12" pad="1"/>
+<wire x1="34.6075" y1="14.82" x2="34.6075" y2="15.875" width="0.3048" layer="1"/>
+<wire x1="34.6075" y1="15.875" x2="35.8775" y2="17.145" width="0.3048" layer="1"/>
+<wire x1="35.8775" y1="17.145" x2="35.8775" y2="19.3675" width="0.3048" layer="1"/>
+<wire x1="35.8775" y1="19.3675" x2="34.29" y2="20.955" width="0.3048" layer="1"/>
+<wire x1="34.29" y1="20.955" x2="33.3375" y2="20.955" width="0.3048" layer="1"/>
 </signal>
 <signal name="N$25">

Commit message: Fixed up previous bugs in offsets
Parts:
- R21: value 5.1k -> 2k
Changed lines of the file:
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@@
 <?xml version="1.0" encoding="utf-8"?>
 <!DOCTYPE eagle SYSTEM "eagle.dtd">
-<eagle version="7.0.0">
+<eagle version="6.5.0">
 <drawing>
 <settings>
@@
 <pass name="Default">
 <param name="RoutingGrid" value="50mil"/>
-<param name="AutoGrid" value="1"/>
-<param name="Efforts" value="0"/>
-<param name="TopRouterVariant" value="1"/>
 <param name="tpViaShape" value="round"/>
 <param name="PrefDir.1" value="|"/>
@@
 <element name="R15" library="rcl" package="R0603" value="3.3k" x="25.0825" y="12.065" rot="R180"/>
 <element name="R16" library="rcl" package="R0603" value="1k" x="26.67" y="13.97"/>
-<element name="R21" library="rcl" package="R0603" value="5.1k" x="29.845" y="13.97"/>
+<element name="R21" library="rcl" package="R0603" value="2k" x="29.845" y="13.97"/>
 <element name="JP1" library="pinhead" package="1X04" value="" x="13.0175" y="6.35"/>
 <element name="JP3" library="pinhead" package="1X04" value="" x="4.1275" y="22.225" rot="R90"/>
